Commit message: Fix Gazebo, RViz, and MoveIt control integration
- stabilize the ROS 2 Docker environment and NVIDIA-backed GUI rendering
- launch Gazebo server and client reliably and bridge simulation time
- raise the UR5e home position and correct ros2_control interfaces
- load MoveIt planning, kinematics, joint limits, and trajectory controllers
- replace the crashing RViz session with a clean motion-planning dashboard
- harden task orchestration and Python package entry-point installation

File: src/ur5e_desk_description/urdf/ur5e_desk.urdf.xacro (robot description, xacro)
@@ -7,5 +7,5 @@
     <visual>
       <geometry>
-        <cylinder radius="0.1" length="0.75"/>
+        <cylinder radius="0.1" length="0.90"/>
       </geometry>
       <material name="dark_gray">
@@ -15,5 +15,5 @@
     <collision>
       <geometry>
-        <cylinder radius="0.1" length="0.75"/>
+        <cylinder radius="0.1" length="0.90"/>
       </geometry>
     </collision>
@@ -27,5 +27,5 @@
     <parent link="world"/>
     <child link="pedestal_link"/>
-    <origin xyz="0.0 -0.5 0.375" rpy="0 0 0"/>
+    <origin xyz="0.0 -0.60 0.45" rpy="0 0 0"/>
   </joint>
   <!-- Include standard UR5e URDF xacro -->
@@ -40,5 +40,5 @@
     visual_parameters_file="$(find ur_description)/config/ur5e/visual_parameters.yaml"
   >
-    <origin xyz="0 0 0.375" rpy="0 0 1.5708"/>
+    <origin xyz="0 0 0.45" rpy="0 0 1.5708"/>
   </xacro:ur_robot>
   <!-- Parallel Jaw Gripper Description -->
@@ -191,9 +191,51 @@
     </plugin>
   </gazebo>
-  <!-- ros2_control interface definition for Gripper -->
-  <ros2_control name="GripperControl" type="system">
+  <!-- One Gazebo hardware system must expose every joint used by controllers. -->
+  <ros2_control name="GazeboSystem" type="system">
     <hardware>
       <plugin>gz_ros2_control/GazeboSimSystem</plugin>
     </hardware>
+    <joint name="shoulder_pan_joint">
+      <command_interface name="position"/>
+      <state_interface name="position">
+        <param name="initial_value">0.0</param>
+      </state_interface>
+      <state_interface name="velocity"/>
+    </joint>
+    <joint name="shoulder_lift_joint">
+      <command_interface name="position"/>
+      <state_interface name="position">
+        <param name="initial_value">-1.5708</param>
+      </state_interface>
+      <state_interface name="velocity"/>
+    </joint>
+    <joint name="elbow_joint">
+      <command_interface name="position"/>
+      <state_interface name="position">
+        <param name="initial_value">1.5708</param>
+      </state_interface>
+      <state_interface name="velocity"/>
+    </joint>
+    <joint name="wrist_1_joint">
+      <command_interface name="position"/>
+      <state_interface name="position">
+        <param name="initial_value">-1.5708</param>
+      </state_interface>
+      <state_interface name="velocity"/>
+    </joint>
+    <joint name="wrist_2_joint">
+      <command_interface name="position"/>
+      <state_interface name="position">
+        <param name="initial_value">-1.5708</param>
+      </state_interface>
+      <state_interface name="velocity"/>
+    </joint>
+    <joint name="wrist_3_joint">
+      <command_interface name="position"/>
+      <state_interface name="position">
+        <param name="initial_value">0.0</param>
+      </state_interface>
+      <state_interface name="velocity"/>
+    </joint>
     <joint name="left_finger_joint">
       <command_interface name="position"/>
@@ -202,7 +244,8 @@
     </joint>
     <joint name="right_finger_joint">
-      <command_interface name="position"/>
       <state_interface name="position"/>
       <state_interface name="velocity"/>
+      <param name="mimic">left_finger_joint</param>
+      <param name="multiplier">1.0</param>
     </joint>
   </ros2_control>
